File: Eagle/V1/Placa/v1.sch (EAGLE design)
At the start: 43 parts

Commit message: v1.0 finalizada
Parts:
- removed AMP, BATERIA, BOTAO, LDR1, LDR2, LED_BATERIA, LED_CONEXAO, MOTORA, MOTORB: (no value), SparkFun-Connectors:CONN_02
- removed HC-SR04: (no value), SparkFun-Connectors:CONN_04
- removed NODEMCU: NODEMCU, nodemcu:NODEMCU
- removed PINOS_DIR, PINOS_ESQ: (no value), SparkFun-Connectors:CONN_07
- removed PINOS_TOPO: (no value), SparkFun-Connectors:CONN_18
- removed PONTEH: TB6612FNG, TB6612FNG:TB6612FNG
- added AE1, AE2, AE3, AE4: (no value), tampi:CONN_03TAMPI
- added AMP2, BAT, CHAVE_PLACA, LDR_DIR, LDR_ESQ, M_A, M_B: (no value), tampi:CONN_02TAMPI
- added BC337: BC337, tampi:BC337
- added DIREITA, ESQUERDA: CONN_07X2TAMPI, tampi:CONN_07X2TAMPI
- added FAROL_FRENTE, FAROL_TRAS, HCSR-04, RGB, SETA_DIR, SETA_ESQ: (no value), tampi:CONN_04
- added R10, R11, R12, R13: (no value), tampi:RESISTOR
- added TAMPA: (no value), tampi:CONN_10X2TAMPI
- added TB6612: TB6612FNGTAMPI, tampi:TB6612FNGTAMPI
- added U$1: NODEMCUTAMPI, tampi:NODEMCUTAMPI
- AMP1: device SparkFun-Connectors:CONN_02 -> tampi:CONN_02TAMPI
- BOOST: value (none) -> MT3608TAMPI; device SparkFun-Connectors:CONN_03 -> tampi:MT3608TAMPI
- BUZZER: value (none) -> BUZZERTAMPI; device SparkFun-Connectors:CONN_02 -> tampi:BUZZERTAMPI
- C1: value 10u -> (none); device capacitor-wima:C2,5-3 -> tampi:CAPACITORTAMPI
- CHARGER: value BATTERY-CHARGER-LI-5V -> TP4056TAMPI; device diy-modules:BATTERY-CHARGER-LI-5V -> tampi:TP4056TAMPI
- CHAVE: device SparkFun-Connectors:CONN_03 -> tampi:CONN_02TAMPI
- IR1, IR2: device SparkFun-Connectors:CONN_04 -> tampi:CONN_04
- IR3, IR4: device SparkFun-Connectors:CONN_04 -> tampi:CONN_03TAMPI
- LED_ON: value (none) -> LEDTAMPI; device SparkFun-Connectors:CONN_02 -> tampi:LEDTAMPI
- MIC: device SparkFun-Connectors:CONN_03 -> tampi:CONN_04
- MUX1, MUX2: device personal:4067_MODULE -> tampi:4067TAMPI
- R1: value 4.7K -> 2.2k; device rcl:R-EU_0204/7 -> tampi:RESISTOR
- R2: value 1.1K -> 1.1k; device rcl:R-EU_0204/7 -> tampi:RESISTOR
- R3: value 2.2K -> (none); device rcl:R-EU_0204/7 -> tampi:RESISTOR
- R4, R5, R8, R9: value 10K -> (none); device rcl:R-EU_0204/7 -> tampi:RESISTOR
- R6, R7: value 100K -> (none); device rcl:R-EU_0204/7 -> tampi:RESISTOR
- SHIFT1, SHIFT2, SHIFT3, SHIFT4, SHIFT5: value 74HC595N -> 74595; device 74xx-eu:74HC595N -> tampi:74595
Connections:
- removed net CHARGER: CHARGER.BAT+, CHAVE.1
- removed net IR1_LED: IR1.3
- removed net IR2_LED: IR2.3
- removed net IR3_LED: IR3.3
- removed net IR4_LED: IR4.3
- removed net LED_BATERIA: R9.2, SHIFT2A.QH
- removed net LED_CONEXAO: R8.2, SHIFT2A.QG
- removed net N$11: MUX2.C12, PINOS_DIR.4
- removed net N$12: MUX2.C11, PINOS_DIR.3
- removed net N$13: MUX2.C10, PINOS_DIR.2
- removed net N$15: MUX2.C8
- removed net N$18: MUX1.C3, PINOS_ESQ.4
- removed net N$19: MUX1.C2, PINOS_ESQ.3
- removed net N$20: MUX1.C1, PINOS_ESQ.2
- removed net N$21: MUX1.C0, PINOS_ESQ.1
- removed net N$22: LED_CONEXAO.2, R8.1
- removed net N$23: LED_BATERIA.2, R9.1
- removed net N$24: MOTORB.2, PONTEH.B2
- removed net N$25: MOTORB.1, PONTEH.B1
- removed net N$26: MOTORA.2, PONTEH.A1
- removed net N$27: MOTORA.1, PONTEH.A2
- removed net N$38: SHIFT1A.QA
- removed net N$46: SHIFT1A.QH
- removed net N$47: SHIFT2A.QA
- new net A1: M_A.1, TB6612.A1
- new net A2: M_A.2, TB6612.A2
- new net AE1: AE1.3, MUX1.C15
- new net AE2: AE2.3, MUX1.C14
- new net AE3: AE3.3, MUX2.C2
- new net AE4: AE4.3, MUX2.C1
- new net B1: M_B.1, TB6612.B1
- new net B2: M_B.2, TB6612.B2
- new net FAROL: FAROL_FRENTE.1, FAROL_FRENTE.4, FAROL_TRAS.1, FAROL_TRAS.4, SHIFT2A.QH
- new net IR_LED_DIR: IR2.3, SHIFT3A.QA
- new net IR_LED_ESQ: IR1.3, SHIFT1A.QA
- new net LD1: DIREITA.12, SHIFT3A.QB
- new net LD2: DIREITA.10, SHIFT3A.QC
- new net LD3: DIREITA.8, SHIFT3A.QD
- new net LD4: DIREITA.6, SHIFT3A.QE
- new net LD5: DIREITA.4, SHIFT3A.QF
- new net LD6: DIREITA.2, SHIFT3A.QG
- new net LE1: ESQUERDA.12, SHIFT1A.QB
- new net LE2: ESQUERDA.10, SHIFT1A.QC
- new net LE3: ESQUERDA.8, SHIFT1A.QD
- new net LE4: ESQUERDA.6, SHIFT1A.QE
- new net LE5: ESQUERDA.4, SHIFT1A.QF
- new net LE6: ESQUERDA.2, SHIFT1A.QG
- new net N$4: R11.1, SETA_ESQ.2, SETA_ESQ.3
- new net RGB_B: R6.2, SHIFT5A.QC
- new net RGB_G: R5.2, SHIFT5A.QB
- new net RGB_R: R4.2, SHIFT5A.QA
- new net SETA_DIR: SETA_DIR.1, SETA_DIR.4, SHIFT3A.QH
- new net SETA_ESQ: SETA_ESQ.1, SETA_ESQ.4, SHIFT1A.QH
- new net TD1: DIREITA.1, MUX2.C15
- new net TD2: DIREITA.3, MUX2.C14
- new net TD3: DIREITA.5, MUX2.C13
- new net TD4: DIREITA.7, MUX2.C12
- new net TD5: DIREITA.9, MUX2.C11
- new net TD6: DIREITA.11, MUX2.C10
- new net TE1: ESQUERDA.11, MUX1.C9
- new net TE2: ESQUERDA.9, MUX1.C8
- new net TE3: ESQUERDA.7, MUX1.C7
- new net TE4: ESQUERDA.5, MUX1.C6
- new net TE5: ESQUERDA.3, MUX1.C5
- new net TE6: ESQUERDA.1, MUX1.C4
- net +3V3: now also AE1.1, AE2.1, AE3.1, AE4.1, DIREITA.14, ESQUERDA.14, IR3.2, IR4.2, MIC.2, SHIFT3P.VCC, SHIFT4P.VCC, SHIFT5P.VCC, TAMPA.17, TB6612.VCC, U$1.3V, U$1.3V@1, U$1.3V@2; no longer BOTAO.1, IR3.4, IR4.4, MIC.1, NODEMCU.3V, NODEMCU.3V@1, NODEMCU.3V@2, PINOS_DIR.1, PINOS_ESQ.7, PINOS_TOPO.6, PONTEH.VCC
- net +5V: now also BOOST.OUT+, BUZZER.2, HCSR-04.4, R7.2, TB6612.VM, U$1.VIN; no longer BOOST.3, HC-SR04.4, NODEMCU.VIN, PONTEH.VM, R5.2
- net +UB: now also BAT.2, CHAVE.2, CHAVE_PLACA.2; no longer AMP.2, AMP1.1, BATERIA.2
- net A0: now also R10.2, U$1.A0; no longer NODEMCU.A0, R1.2
- net AIN1: now also SHIFT5A.QE, TB6612.AIN1; no longer PONTEH.AIN1, SHIFT2A.QC
- net AIN2: now also SHIFT5A.QD, TB6612.AIN2; no longer PONTEH.AIN2, SHIFT2A.QB
- net BAT: now also MUX1.C1, R8.1; no longer MUX1.C11, R6.1, R7.2
- net BIN1: now also SHIFT5A.QG, TB6612.BIN1; no longer PONTEH.BIN1, SHIFT2A.QE
- net BIN2: now also SHIFT5A.QH, TB6612.BIN2; no longer PONTEH.BIN2, SHIFT2A.QF
- net BOOST: now also BOOST.IN+, CHARGER.OUT+, R8.2; no longer BOOST.1, CHAVE.3, R6.2
- net BOTAO: now also R3.1, TAMPA.19, U$1.D1; no longer BOTAO.2, NODEMCU.D1, PINOS_TOPO.5, R4.1
- net BUZZER: now also R13.1, U$1.D0; no longer BUZZER.2, NODEMCU.D0
- net CLK: now also U$1.D7; no longer NODEMCU.D7
- net DATA: now also U$1.D5; no longer NODEMCU.D5
- net ECHO: now also HCSR-04.2; no longer HC-SR04.2
- net EN1: now also SHIFT2A.QF; no longer SHIFT1A.QF
- net EN2: now also SHIFT2A.QG; no longer SHIFT1A.QG
- net GND: now also AE1.2, AE2.2, AE3.2, AE4.2, BAT.1, BC337.E, BOOST.IN-, BOOST.OUT-, CHARGER.B-, CHARGER.OUT-, HCSR-04.1, LDR_DIR.1, LDR_ESQ.1, LED_ON.C, MIC.3, R10.1, R11.2, R12.2, R3.2, R9.2, RGB.3, SHIFT3P.GND, SHIFT4P.GND, SHIFT5P.GND, TB6612.GND1, TB6612.GND2, TB6612.GND3, U$1.GND@2, U$1.GND@3, U$1.GND@4; no longer BATERIA.1, BOOST.2, BUZZER.1, CHARGER.BAT-, HC-SR04.1, LDR1.1, LDR2.1, LED_BATERIA.1, LED_CONEXAO.1, LED_ON.1, MIC.2, NODEMCU.GND@2, NODEMCU.GND@3, NODEMCU.GND@4, PONTEH.GND1, PONTEH.GND2, PONTEH.GND3, R3.1, R4.2, R7.1
- net IR1_SEN: now also MUX1.C3; no longer MUX1.C9
- net IR2_SEN: now also IR4.3, MUX2.C8; no longer IR2.2, MUX2.C6
- net IR3_SEN: now also IR3.3, MUX1.C2; no longer IR3.2, MUX1.C8
- net IR4_SEN: now also IR2.2; no longer IR4.2
- net L1: now also SHIFT4A.QH, TAMPA.1; no longer PINOS_TOPO.7, SHIFT5A.QH
- net L2: now also SHIFT4A.QG, TAMPA.3; no longer PINOS_TOPO.8, SHIFT5A.QG
- net L3: now also SHIFT4A.QF, TAMPA.5; no longer PINOS_TOPO.9, SHIFT5A.QF
- net L4: now also SHIFT4A.QE, TAMPA.7; no longer PINOS_TOPO.10, SHIFT5A.QE
- net L5: now also SHIFT4A.QD, TAMPA.9; no longer PINOS_TOPO.11, SHIFT5A.QD
- net L6: now also SHIFT4A.QC, TAMPA.11; no longer PINOS_TOPO.12, SHIFT5A.QC
- net L7: now also SHIFT4A.QB, TAMPA.13; no longer PINOS_TOPO.13, SHIFT5A.QB
- net L8: now also SHIFT4A.QA, TAMPA.15; no longer PINOS_TOPO.14, SHIFT5A.QA
- net LATCH: now also U$1.D6; no longer NODEMCU.D6
- net LDR1: now also LDR_ESQ.2, MUX1.C0; no longer LDR1.2, MUX1.C10
- net LDR2: now also LDR_DIR.2, MUX2.C9; no longer LDR2.2, MUX2.C5
- net MIC: now also MIC.4, MUX2.C0; no longer MIC.3, MUX2.C4
- net N$1: now also R4.1, RGB.4; no longer MUX1.C6
- net N$10: now also BC337.C, BUZZER.1; no longer MUX2.C13, PINOS_DIR.5
- net N$2: now also R5.1, RGB.2; no longer MUX2.C9
- net N$28: now also LED_ON.A, R7.1; no longer LED_ON.2, R5.1
- net N$29: now also SHIFT3A.QH*; no longer SHIFT4A.QH*
- net N$3: now also R6.1, RGB.1; no longer MUX1.C7
- net N$30: now also SHIFT3A.SER, SHIFT4A.QH*; no longer SHIFT3A.QH*, SHIFT4A.SER
- net N$31: now also SHIFT4A.SER; no longer SHIFT3A.SER
- net N$39: now also R1.2, U$1.D2; no longer NODEMCU.D2, R3.2
- net N$6: now also FAROL_FRENTE.2, FAROL_FRENTE.3, FAROL_TRAS.2, FAROL_TRAS.3, R9.1; no longer MUX1.C5, PINOS_ESQ.6
- net N$7: now also R12.1, SETA_DIR.2, SETA_DIR.3; no longer MUX1.C4, PINOS_ESQ.5
- net N$8: now also AMP1.2, AMP2.2, CHAVE.1, CHAVE_PLACA.1; no longer MUX2.C15, PINOS_DIR.7
- net N$9: now also BC337.B, R13.2; no longer MUX2.C14, PINOS_DIR.6
- net PWMA: now also TB6612.PWMA, U$1.D4; no longer NODEMCU.D8, PONTEH.PWMA
- net PWMB: now also TB6612.PWMB, U$1.D8; no longer NODEMCU.D4, PONTEH.PWMB
- net S0: now also SHIFT2A.QE; no longer SHIFT1A.QE
- net S1: now also SHIFT2A.QD; no longer SHIFT1A.QD
- net S2: now also SHIFT2A.QC; no longer SHIFT1A.QC
- net S3: now also SHIFT2A.QB; no longer SHIFT1A.QB
- net STBY: now also SHIFT5A.QF, TB6612.STBY; no longer PONTEH.STBY, SHIFT2A.QD
- net T1: now also MUX1.C10, TAMPA.8; no longer MUX1.C12, PINOS_TOPO.1
- net T2: now also MUX1.C11, TAMPA.6; no longer MUX1.C13, PINOS_TOPO.2
- net T3: now also MUX1.C12, TAMPA.4; no longer MUX1.C14, PINOS_TOPO.3
- net T4: now also MUX1.C13, TAMPA.2; no longer MUX1.C15, PINOS_TOPO.4
- net T5: now also MUX2.C3, TAMPA.20; no longer MUX2.C0, PINOS_TOPO.15
- net T6: now also MUX2.C4, TAMPA.18; no longer MUX2.C1, PINOS_TOPO.16
- net T7: now also MUX2.C5, TAMPA.16; no longer MUX2.C2, PINOS_TOPO.17
- net T8: now also MUX2.C6, TAMPA.14; no longer MUX2.C3, PINOS_TOPO.18
- net TRIG: now also HCSR-04.3, U$1.D3; no longer HC-SR04.3, NODEMCU.D3
- net VAMP: now also AMP1.1, AMP2.1, CHARGER.B+; no longer AMP.1, AMP1.2, CHAVE.2
Other:
- moved on the sheet: BUZZER, CHARGER, R1, R3, R4, R5, R6, R7, R8, R9, SHIFT1P, SHIFT2P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
