File: Eagle/V1/Trilhas maiores/v1.brd (EAGLE design)
At the start: 100 x 100 mm, 55 parts

Commit message: gerber files
Routing:
- net N$8: track 31.1 -> 20.3 mm, vias 2 -> 0
- net LD4: track 45.7 -> 48.3 mm
- net +UB: track 27.2 -> 24.8 mm
- net DATA: track 55.4 -> 57.1 mm
- net LD6: track 41.8 -> 42.4 mm
- net LD3: track 59.2 -> 59.8 mm
- added copper zone on layer 1, net GND
- added copper zone on layer 16, net GND
